File: sensor_board.kicad_sch (KiCad schematic)
At the start: 44 parts, among them IC1 INA826AID, J1 JST-GH, J2 JST-GH, J3 Conn_01x02_Socket, J5 Conn_01x04_Socket, U2 MCP6001-OT, U3 MIC5504-3.3YM5, U4 ADC101C021CIMM

Commit message: cleanup and export 3d models
Other:
- company: (none) -> TUDSaT
- title: (none) -> Sensor Board
